Commit message: Add missing camera-rgbd-frame link

File: urdf/r2d2_bot.xacro (robot description, xacro)
@@ -261,3 +261,9 @@
     <parent link="chassis"/>
   </joint>
+  <link name="camera_rgbd_frame"></link>
+  <joint name="camera_rgbd_joint" type="fixed">
+    <origin xyz="0 0 0" rpy="-${pi/2} 0 -${pi/2}"/>
+    <parent link="camera"/>
+    <child link="camera_rgbd_frame"/>
+  </joint>
 </robot>
